Commit message: feat: 配置项目环境和修复编译问题
- 更新 VS Code 配置以支持 clangd
- 为所有包添加 CMAKE_EXPORT_COMPILE_COMMANDS
- 修复启动脚本的 set -u 问题
- 添加新功能包: sentry_control, sentry_nav_decision_interface, serial, auto_aim_interfaces
- 修复 UTF-8 编码问题
- 更新配置文件和启动脚本

File: src/rm_nav_bringup/urdf/sentry_robot_real.xacro (robot description, xacro)
@@ -132,4 +132,5 @@
     <visual>
       <origin xyz="0.025 -0.0265 -0.025" rpy="${pi/2} 0 ${pi}"/>
+      <!-- <origin xyz="0.025 -0.0265 -0.025" rpy="0 0 ${pi}"/> -->
       <geometry>
         <mesh filename="package://pb_rm_simulation/meshes/mid360.stl" scale="0.001 0.001 0.001"/>
